Commit message: fabrica.beam_2x: coarse-receptive URDFs (hole CoACD + bulk boxes) + skill
Switch beam_2x receptives to the same recipe used for fmb.peg_board_1: only
the receiver's CoACD hulls that overlap the inserter's A-frame bbox (with
5mm padding) are kept as fine-collision <mesh>; the rest of the receiver is
replaced by a 4-box frame around the hole region (clipped to the receiver's
A-frame bbox); each non-receiver fixture part collapses to a single
A-frame-aligned <box> primitive.

Receivers vary per problem (inserts_into = {2:6, 0:2, 3:6, 1:3}), so the
classification runs per-problem and writes one URDF per inserter at
insertion_fixtures/part_<inserter>.urdf, replacing the previous
"every-fixture-part-fully-CoACD'd" output.

problems.py keeps the legacy code path as a fallback for assemblies whose
receptive URDFs haven't been pre-generated, but uses the new pre-generated
URDFs whenever they exist on disk.

Also adds a Claude skill at
.claude/skills/insertion-problem-from-coarse-receptive/SKILL.md that
documents the whole pipeline (Recipe A for FMB peg-in-hole boards, Recipe B
for fabrica-style multi-part fixtures), the gotchas (manifold3d for
slicing, CoACD-only never V-HACD, max_convex_hull cap, canonical-rotation
flag), and the canonical implementation file map.

Co-Authored-By: Claude Opus 4.7 (1M context) <noreply@anthropic.com>

File: assets/urdf/fabrica/beam_2x/insertion_fixtures/part_0.urdf (robot description, URDF)
Before this commit: robot fixture_beam_2x_part_0, 3 links, 2 joints
Links:
- removed link part_2
- removed link part_6
- removed link root
- added link plate; collision box size=0.304800 0.035560 0.025400; collision mesh filename=../2/coacd/decomp_0.obj scale=1 1 1
Joints:
- removed joint root_to_part_2
- removed joint root_to_part_6

File: assets/urdf/fabrica/beam_2x/insertion_fixtures/part_1.urdf (robot description, URDF)
Before this commit: robot fixture_beam_2x_part_1, 5 links, 4 joints
Links:
- removed link part_0
- removed link part_2
- removed link part_3
- removed link part_6
- removed link root
- added link plate; collision box size=0.023006 0.024007 0.152400; collision box size=0.025400 0.152400 0.030480
Joints:
- removed joint root_to_part_0
- removed joint root_to_part_2
- removed joint root_to_part_3
- removed joint root_to_part_6

File: assets/urdf/fabrica/beam_2x/insertion_fixtures/part_2.urdf (robot description, URDF)
Before this commit: robot fixture_beam_2x_part_2, 2 links, 1 joints
Links:
- removed link part_6
- removed link root
- added link plate; collision box size=0.051994 0.024007 0.025400; collision box size=0.229800 0.024007 0.025400
Joints:
- removed joint root_to_part_6

File: assets/urdf/fabrica/beam_2x/insertion_fixtures/part_3.urdf (robot description, URDF)
Before this commit: robot fixture_beam_2x_part_3, 4 links, 3 joints
Links:
- removed link part_0
- removed link part_2
- removed link part_6
- removed link root
- added link plate; collision box size=0.023006 0.024007 0.152400; collision box size=0.025400 0.152400 0.030480
Joints:
- removed joint root_to_part_0
- removed joint root_to_part_2
- removed joint root_to_part_6
