Commit message: fmb hybrid: tip = board thickness (50mm), pre_insert_offset = 50mm
The fmb peg-in-hole boards are 50mm thick. The previous defaults
(tip = 25mm, pre_insert_offset = 40mm) under-covered the hole. Bumped
both to match the board thickness so the SDF tip spans the full hole
depth at insertion and the pre-insert hover sits exactly one
board-thickness above the hole entrance.

Files:
  fmb/peg_board_problem_setup/step3_generate_sdf_hybrid.py
    TIP_HEIGHT_M 0.025 → 0.05.
  fmb/problems.py
    pre_insert_offset 0.04 → 0.05 for both base and hybrid Problems
    on peg_board_1.
  All 9 fmb peg_<N>/sdf_hybrid/ assets regenerated (tip + body OBJs
    + body CoACD hulls + hybrid URDFs).

Add the missing table to validate_insertions.py: previously the
script only added a ground plane, so any inserter that fell out of
the receptive's hole dropped 53 cm to the floor and the settle_kp
metric blew up by ~ TABLE_TOP_Z. Now we also create_actor a
fix-base box matching the env's table_narrow.urdf at world (0, 0,
TABLE_RESET_Z). The descent kp_max is unchanged; the settle_kp is
now meaningful for fmb peg-board problems where there's just a few
mm of clearance and the peg can pop out without a robot holding it.

Add fmb_peg_board_1_peg_46_sdf_hybrid_better_physics finetune_rgf10
.sub mirroring the fabrica better_physics one — same SDF-friendly
PhysX overrides (num_position_iterations 32, num_velocity_iterations 1,
bounce_threshold_velocity 0.05, max_depenetration_velocity 10.0,
friction_offset_threshold 0.01, friction_correlation_distance 0.0005),
just pointed at fmb.peg_board_1.peg_46_sdf_hybrid.

Co-Authored-By: Claude Opus 4.7 (1M context) <noreply@anthropic.com>

File: assets/urdf/fmb/pegs/peg_31/sdf_hybrid/peg_31_sdf_hybrid.urdf (robot description, URDF)
Before this commit: robot fmb_peg_31_sdf_hybrid, 3 links, 2 joints
Links:
- link body_link: geometry collision mesh filename=coacd/decomp_0.obj scale=1 1 1; collision mesh filename=coacd/decomp_1.obj scale=1 1 1

File: assets/urdf/fmb/pegs/peg_36/sdf_hybrid/peg_36_sdf_hybrid.urdf (robot description, URDF)
Before this commit: robot fmb_peg_36_sdf_hybrid, 3 links, 2 joints
Links:
- link body_link: geometry collision mesh filename=coacd/decomp_0.obj scale=1 1 1; collision mesh filename=coacd/decomp_1.obj scale=1 1 1

File: assets/urdf/fmb/pegs/peg_40/sdf_hybrid/peg_40_sdf_hybrid.urdf (robot description, URDF)
Before this commit: robot fmb_peg_40_sdf_hybrid, 3 links, 2 joints
Links:
- link body_link: geometry collision mesh filename=coacd/decomp_0.obj scale=1 1 1; collision mesh filename=coacd/decomp_1.obj scale=1 1 1
