Commit message: Update FMB canonical peg assets

File: assets/urdf/fmb/pegs/peg_31/coacd/peg_31_coacd.urdf (robot description, URDF)
Before this commit: robot peg_31_coacd, 10 links, 9 joints
Links:
- added link hull_9, mass 0.001; collision mesh filename=decomp_9.obj scale=1 1 1; visual mesh filename=decomp_9.obj scale=1 1 1
Joints:
- added joint hull_joint_9: type fixed, parent base_link, child hull_9, origin xyz=0 0 0 rpy=0 0 0

File: assets/urdf/fmb/pegs/peg_31/sdf_hybrid/peg_31_sdf_hybrid.urdf (robot description, URDF)
Before this commit: robot fmb_peg_31_sdf_hybrid, 3 links, 2 joints
Links:
- link body_link: geometry collision mesh filename=coacd/decomp_0.obj scale=1 1 1; collision mesh filename=coacd/decomp_1.obj scale=1 1 1

File: assets/urdf/fmb/pegs/peg_36/coacd/peg_36_coacd.urdf (robot description, URDF)
Before this commit: robot peg_36_coacd, 6 links, 5 joints
Links:
- removed link hull_4
Joints:
- removed joint hull_joint_4

File: assets/urdf/fmb/pegs/peg_36/sdf_hybrid/peg_36_sdf_hybrid.urdf (robot description, URDF)
Before this commit: robot fmb_peg_36_sdf_hybrid, 3 links, 2 joints
Links:
- link body_link: geometry collision mesh filename=coacd/decomp_0.obj scale=1 1 1; collision mesh filename=coacd/decomp_1.obj scale=1 1 1
