Commit message: Add play2win problems, asset regeneration, env fixes
* peg: Lpeg (one-sided L-shaped head) variant + problem registration
* fabrica beam_2x: tip axis chosen by insertion direction (not longest
  extent), Z-aware bulk decomposition, tip clipped to receiver footprint
* furniture_bench one_leg: open-top tray (4 walls + base plate) fixture
* furniture_bench bulb_screw: full step1/2/3 pipeline + lamp.py upstream
  snapshot, R_x(-90) flipped receiver, base box + SDF socket fixture,
  CoACD-decomposed bulb body, separate visualize_bulb_threading viewer
* PegInHole env: stop hard-coding identity start orientation; defer to
  SimToolReal _reset_object_pose so reset_position_noise + random_orientation
  actually apply (eval_isaacsim no longer zeroes them)
* visualize_problems: hole_y_range narrowed to [-0.1, 0.1]; fixture
  variation footprint + assembly XY sliders
* play2win/: 7 finetune .sub files (peg_insertion, multi_part_assembly,
  furniture_screwing) at 200 GB mem, screwing tols 5/2 mm,
  peg+assembly tols 10/5 mm

Co-Authored-By: Claude Opus 4.7 (1M context) <noreply@anthropic.com>

File: assets/urdf/fabrica/beam_2x/0/sdf_hybrid/beam_2x_0_sdf_hybrid.urdf (robot description, URDF)
Before this commit: robot beam_2x_0_sdf_hybrid, 3 links, 2 joints
Links:
- link body_link: geometry collision mesh filename=coacd/decomp_0.obj scale=1 1 1; collision mesh filename=coacd/decomp_1.obj scale=1 1 1

File: assets/urdf/fabrica/beam_2x/2/sdf_hybrid/beam_2x_2_sdf_hybrid.urdf (robot description, URDF)
Before this commit: robot beam_2x_2_sdf_hybrid, 3 links, 2 joints
Links:
- link body_link: geometry collision mesh filename=coacd/decomp_0.obj scale=1 1 1; collision mesh filename=coacd/decomp_1.obj scale=1 1 1

File: assets/urdf/fabrica/beam_2x/insertion_fixtures/part_0_sdf_hybrid.urdf (robot description, URDF)
Before this commit: robot fixture_beam_2x_part_0_sdf_hybrid, 1 links, 0 joints
Links:
- link plate: geometry collision box size=0.023006 0.024007 0.127000; collision box size=0.304800 0.035560 0.025400

File: assets/urdf/furniture_bench/square_table/insertion_fixtures/one_leg_sdf_hybrid.urdf (robot description, URDF)
Before this commit: robot one_leg_receptive_sdf_hybrid, 1 links, 0 joints
Links:
- link receptive: geometry collision box size=0.005000 0.152501 0.026250; collision box size=0.005000 0.152501 0.026250
