Commit message: matched-mass URDFs + furniture_bench 2x/1.5x clones + leg collision fixes
Asset physics modeling for the fig2 panel-(a) tasks (PegInHole, Fabrica
Beam, FurnitureBench leg-screwing). Two findings drove this:

  1. Isaac Sim's URDF importer silently drops <density> tags; URDFs that
     relied on it (fabrica beam_3x parts) were effectively running with
     placeholder mass. Replaced with explicit <mass>+<inertia> using
     measured part masses + mesh-derived inertia tensors.
  2. visualize_problems renders <visual>, not <collision>; cylinder /
     sphere primitives weren't supported. Added support to the loader
     so capsule-style hole approximations show up in viser.

Furniture bench (one_leg task):

  * scene_generation/scale_one_leg.py: new scaler that rewrites OBJ
    vertices by --scale, renames part dirs/files, scales URDF xyz / box
    size / cylinder radius+length, and scales JSON length fields. Used
    to mint square_table_1p5x and square_table_2x clones (legs+top+
    hole_patches+insertion_fixtures+setup JSONs).
  * square_table_leg4: CoACD-decomposed the body mesh into 12 hulls
    (body_coacd/decomp_*.obj). SDF-hybrid URDF now has per-hull
    visual+collision pairs for the body (mirroring fabrica/beam_3x
    convention) and keeps SDF on the threaded tip.
  * Matched-mass leg URDFs (CoACD + SDF-hybrid variants) at 1x/1.5x/2x:
      1x   measured 22.75 g  ρ≈318 kg/m³
      1.5x measured 63.97 g  ρ≈265 kg/m³ (hull V; ≈304 filled)
      2x   151.84 g          placeholder, replace when weighed
  * one_leg.urdf fixture: visual swapped synthetic slab -> canonical
    mesh so all 4 hole geometries are rendered; cylinder collisions at
    the 3 inactive corners (redundant with bulk boxes but reserved for
    future swiss-cheese carve).
  * one_leg_sdf_hybrid.urdf fixture: added 3 r=16 mm cylinder visual+
    collision pairs at the inactive corners (matching the active hole-
    detail mesh footprint), so all 4 holes are visible.
  * furniture_bench/objects.py: discover *_matchedmass_coacd and
    *_matchedmass_sdf_hybrid siblings; PIECES now includes
    square_table_1p5x and square_table_2x.
  * furniture_bench/problems.py: _register_one_leg() parameterized on
    piece + problem_suffix; registers 1x, 1.5x, 2x variants, each with
    matched-mass siblings for CoACD and SDF-hybrid.

Fabrica (beam_3x):

  * beam_3x parts 0/1/2/3 (and 6 as fixture-only placeholder): matched-
    mass URDFs at the mesh, CoACD, and SDF-hybrid level, all patched
    via base_link <inertial> with measured mass:
      part 0,1 -> 85.98 g  ρ≈309 kg/m³
      part 2,3 -> 68.57 g  ρ≈335 kg/m³
      part 6   -> 82.50 g  placeholder (fixture-only)
  * fabrica/objects.py: discover *_matchedmass_sdf_hybrid siblings.
  * fabrica/problems.py: register part_N_matchedmass (CoACD) and
    part_N_matchedmass_sdf_hybrid problem variants.

Diagnostic + helpers:

  * debug_differences/smoke_urdf_density_inertia.py: probe how
    UrdfConverter+PhysX handle the four ways of specifying inertial
    (density-only, mass-only, mass+inertia, missing block).
  * assets/urdf/furniture_bench/square_table/square_table_leg4/
    square_table_leg4_canonical.stl: 1x leg STL for measurement.

Co-Authored-By: Claude Opus 4.7 (1M context) <noreply@anthropic.com>

File: assets/urdf/furniture_bench/square_table/insertion_fixtures/one_leg.urdf (robot description, URDF)
Before this commit: robot one_leg_receptive, 1 links, 0 joints
Links:
- link receptive: geometry collision box size=0.014607999999999996 0.01998699999999999 0.03125; collision box size=0.127108 0.01998699999999999 0.03125

File: assets/urdf/furniture_bench/square_table/insertion_fixtures/one_leg_sdf_hybrid.urdf (robot description, URDF)
Before this commit: robot one_leg_receptive_sdf_hybrid, 1 links, 0 joints
Links:
- link receptive: geometry collision box size=0.005000 0.152501 0.026250; collision box size=0.005000 0.152501 0.026250

File: assets/urdf/furniture_bench/square_table/square_table_leg4/sdf_hybrid/square_table_leg4_sdf_hybrid.urdf (robot description, URDF)
Before this commit: robot square_table_leg4_sdf_hybrid, 3 links, 2 joints
Links:
- link body_link: geometry collision mesh filename=body_coacd/decomp_0.obj scale=1 1 1; collision mesh filename=body_coacd/decomp_1.obj scale=1 1 1
